File: m0110a.kicad_pcb (KiCad board)
At the start: 2 copper layers, 365.1 x 97.6 mm, 159 parts, among them U1 Teensy2.0_(C)

Commit message: connect third and fourth row diodes and rgb data lines
Parts:
- moved D70 2.35 mm to (342.1, 56.4)
- moved D37 1.04 mm to (259.3, 39.1)
- moved D42 0.34 mm to (136.3, 39.1)
- moved D60 0.34 mm to (145.8, 58.2)
- moved D62 0.34 mm to (183.9, 58.2)
- moved D58 0.34 mm to (107.7, 58.2)
- moved D59 0.34 mm to (126.7, 58.2)
- moved D38 0.34 mm to (212.5, 39.1)
- moved D55 0.34 mm to (222.0, 58.2)
- moved D61 0.34 mm to (164.8, 58.2)
- moved D67 0.34 mm to (202.9, 58.2)
- moved D63 0.31 mm to (243.5, 58.2)
- moved D68 0.30 mm to (313.4, 58.2)
- moved D69 0.29 mm to (264.9, 58.2)
- moved D47 0.26 mm to (174.5, 39.1)
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Routing:
- net ROW2: track 0.00 -> 335.8 mm
- net ROW3: track 0.00 -> 321.3 mm
- net Net-(MX63-Pad5): track 0.00 -> 38.5 mm
- net Net-(MX44-Pad4): track 0.00 -> 32.3 mm
- net Net-(MX66-Pad4): track 0.00 -> 26.4 mm
- net Net-(MX61-Pad5): track 0.00 -> 25.2 mm
- net Net-(MX47-Pad5): track 0.00 -> 21.6 mm
- net Net-(MX51-Pad4): track 0.00 -> 21.6 mm
- net Net-(MX59-Pad5): track 0.00 -> 16.9 mm
- net Net-(MX61-Pad4): track 0.00 -> 16.9 mm
- net Net-(MX63-Pad4): track 0.00 -> 14.5 mm
- net Net-(MX62-Pad5): track 0.00 -> 14.5 mm
- net Net-(MX54-Pad5): track 0.00 -> 14.5 mm
- net Net-(MX45-Pad4): track 0.00 -> 14.5 mm
- net Net-(MX44-Pad5): track 0.00 -> 14.5 mm
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
Commit message: add column connections
Parts:
- moved U1 0.41 mm to (94.6, 76.6)
- moved D71 0.22 mm to (134.1, 77.2)
- moved D72 0.22 mm to (332.6, 77.2)
- moved D73 0.22 mm to (55.6, 77.2)
- moved D74 0.22 mm to (227.0, 77.2)
- moved D75 0.22 mm to (15.1, 77.2)
- moved D76 0.22 mm to (208.0, 77.2)
- moved D77 0.22 mm to (246.1, 77.2)
- moved D78 0.22 mm to (305.6, 77.2)
- moved D79 0.22 mm to (265.1, 77.2)
Connections:
- MX55 pad 1: Net-(MX55-Pad1) -> COL5
- MX55 pad 3: COL5 -> Net-(MX55-Pad3)
- MX68 pad 1: COL12 -> COL11
- MX72 pad 1: COL10 -> COL9
- MX74 pad 1: COL11 -> COL10
- MX78 pad 1: COL12 -> COL11
- U1 pad 17: Net-(U1-Pad17) -> ROW4
Routing:
- net ROW4: track 0.00 -> 319.8 mm
- net COL10: track 0.00 -> 104.3 mm, vias 0 -> 5
- net COL9: track 0.00 -> 103.3 mm, vias 0 -> 5
- net COL11: track 0.00 -> 102.6 mm, vias 0 -> 5
- net COL5: track 0.00 -> 102.2 mm, vias 0 -> 5
- net COL13: track 0.00 -> 99.0 mm, vias 0 -> 5
- net COL14: track 0.00 -> 98.7 mm, vias 0 -> 5
- net COL1: track 0.00 -> 97.3 mm, vias 0 -> 5
- net COL0: track 0.00 -> 96.9 mm, vias 0 -> 5
- net COL17: track 0.00 -> 94.8 mm, vias 0 -> 4
- net COL16: track 0.00 -> 89.8 mm, vias 0 -> 5
- net COL3: track 0.00 -> 78.5 mm, vias 0 -> 4
- net COL6: track 0.00 -> 76.9 mm, vias 0 -> 4
- net COL8: track 0.00 -> 76.8 mm, vias 0 -> 4
- net COL4: track 0.00 -> 76.2 mm, vias 0 -> 4
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