File: m0110a.kicad_pcb (KiCad board)
At the start: 2 copper layers, 177 parts, among them SW1 SW_Push, U1 ATmega32U4-AU, Y1 16MHz

Commit message: place main alpha numeric section
Parts:
- moved MX_BSLSH1 343.4 mm to (257.2, 19.1)
- moved MX_A1 340.5 mm to (33.3, 38.1)
- moved MX_L1 320.2 mm to (185.7, 38.1)
- moved MX_RSFT1 319.6 mm to (235.7, 57.1)
- moved MX_P1 310.4 mm to (200.0, 19.1)
- moved MX_D1 304.7 mm to (71.4, 38.1)
- moved MX_K1 297.0 mm to (166.7, 38.1)
- moved MX_RIGHT1 291.8 mm to (257.2, 76.2)
- moved MX_B1 291.7 mm to (119.1, 57.1)
- moved MX_C1 283.3 mm to (81.0, 57.1)
- moved MX_I1 280.5 mm to (161.9, 19.1)
- moved MX_J1 280.3 mm to (147.6, 38.1)
- moved MX_SEMI1 279.9 mm to (204.8, 38.1)
- moved MX_Z1 279.8 mm to (42.9, 57.1)
- moved MX_N1 278.7 mm to (138.1, 57.1)
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
Commit message: placed number pad
Parts:
- U1: moved to B.Cu
- moved MX_NUM_SLSH1 403.0 mm to (325.4, 0.00)
- moved MX_NUM_MUL1 389.9 mm to (344.5, 0.00)
- moved MX_NUM_ADD1 351.7 mm to (344.5, 38.1)
- moved MX_NUM_7 346.0 mm to (287.3, 19.1)
- moved MX_NUM_5 332.7 mm to (306.4, 38.1)
- moved MX_NUM_DOT1 302.3 mm to (325.4, 76.2)
- moved MX_NUM_2 292.8 mm to (306.4, 57.1)
- moved MX_NUM_9 282.1 mm to (325.4, 19.1)
- moved MX_NUM_3 275.8 mm to (325.4, 57.1)
- moved MX_NUM_EQL1 263.5 mm to (306.4, 0.00)
- moved MX_NUM_BIG_0 260.1 mm to (296.9, 76.2)
- moved MX_NUM_MINS1 255.9 mm to (344.5, 19.1)
- moved MX_NUM_8 235.8 mm to (306.4, 19.1)
- moved MX_NUM_4 224.7 mm to (287.3, 38.1)
- moved MX_NUM_ENT1 215.8 mm to (344.5, 66.7), turned to 90 degrees
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
Commit message: start placing controller footprints
Parts:
- C1, C2, C3, C4, C5, C6, C7, D1, D10, D11, D12, D13, D14, D15, D16, D17, D18, D19, D2, D20, D21, D22, D23, D24, D25, D26, D27, D28, D29, D3, D30, D31, D32, D33, D34, D35, D36, D37, D38, D39, D4, D40, D41, D42, D43, D44, D45, D46, D47, D48, D49, D5, D50, D51, D52, D53, D54, D55, D56, D57, D58, D59, D6, D60, D61, D62, D63, D64, D65, D66, D67, D68, D69, D7, D70, D71, D72, D73, D74, D75, D76, D77, D78, D79, D8, D80, D9, F1, R1, R2, R3, R4, SW1, USB1, Y1: moved to B.Cu
- moved D53 308.3 mm to (352.4, 38.9), turned to 90 degrees
- moved D18 300.3 mm to (352.4, 0.79), turned to 90 degrees
- moved D36 289.7 mm to (352.4, 19.8), turned to 90 degrees
- moved D70 288.9 mm to (339.7, 59.5), turned to 270 degrees
- moved D73 279.7 mm to (331.0, 69.8), turned to 270 degrees
- moved D51 279.4 mm to (314.3, 38.9), turned to 90 degrees
- moved D1 278.3 mm to (7.94, 0.79), turned to 90 degrees
- moved USB1 270.5 mm to (272.3, -7.94), turned to 270 degrees
- moved D19 265.6 mm to (12.7, 19.8), turned to 90 degrees
- moved D20 264.0 mm to (36.5, 19.8), turned to 90 degrees
- moved D5 260.7 mm to (84.1, 0.79), turned to 90 degrees
- moved D2 259.5 mm to (27.0, 0.79), turned to 90 degrees
- moved D6 258.3 mm to (103.2, 0.79), turned to 90 degrees
- moved D37 256.2 mm to (15.1, 38.9), turned to 90 degrees
- moved D3 252.2 mm to (46.0, 0.79), turned to 90 degrees
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
Commit message: connect chematic. start placing footprints
Parts:
- removed C1, C2: 22pF, Capacitor_SMD:C_0805_2012Metric
- removed C3: 1uF, Capacitor_SMD:C_0805_2012Metric
- removed C4, C5, C6: 0.1uF, Capacitor_SMD:C_0805_2012Metric
- removed C7: 10uF, Capacitor_SMD:C_0805_2012Metric
- removed D80: D_Small, Diode_SMD:D_SOD-123
- removed F1: 500mA, Fuse:Fuse_1206_3216Metric
- removed MX_1, MX_2, MX_3, MX_4, MX_5, MX_6, MX_7, MX_8, MX_9, MX_A1, MX_B1, MX_BSLSH1, MX_C1, MX_COMMA1, MX_D1, MX_DOT1, MX_DWN1, MX_E1, MX_EQL1, MX_ESC1, MX_F1, MX_FN1, MX_G1, MX_H1, MX_I1, MX_J1, MX_K1, MX_L1, MX_LBRC1, MX_LEFT1, MX_M1, MX_MINS1, MX_N1, MX_NUM1, MX_NUM_0, MX_NUM_1, MX_NUM_2, MX_NUM_3, MX_NUM_4, MX_NUM_5, MX_NUM_6, MX_NUM_7, MX_NUM_8, MX_NUM_9, MX_NUM_ADD1, MX_NUM_DBL_0, MX_NUM_DOT1, MX_NUM_EQL1, MX_NUM_MINS1, MX_NUM_MUL1, MX_NUM_SLSH1, MX_O1, MX_P1, MX_Q1, MX_QUOT1, MX_R1, MX_RBRC1, MX_RIGHT1, MX_S1, MX_SEMI1, MX_SLSH1, MX_T1, MX_U1, MX_UP1, MX_V1, MX_W1, MX_X1, MX_Y1, MX_Z1, MX_ZERO1: MX-LED, MX_Alps_Hybrid:MX-1U
- removed MX_7U_SPC1: MX-LED, MX_Alps_Hybrid:MX-7U
- removed MX_BSPC1, MX_LALT1, MX_TAB1: MX-LED, MX_Alps_Hybrid:MX-1.5U
- removed MX_CAP1, MX_ENTER1: MX-LED, MX_Alps_Hybrid:MX-1.75U
- removed MX_LGUI1, MX_NUM_BIG_0, MX_NUM_ENT1: MX-LED, MX_Alps_Hybrid:MX-2U
- removed MX_LSFT1: MX-LED, MX_Alps_Hybrid:MX-2.25U
- removed MX_RSFT1: MX-LED, MX_Alps_Hybrid:MX-1.25U
- removed R1, R4: 10k, Resistor_SMD:R_0805_2012Metric
- removed R2, R3: 22, Resistor_SMD:R_0805_2012Metric
- removed USB1: Molex-0548190589, random-keyboard-parts:Molex-0548190589
- removed Y1: 16MHz, Crystal:Crystal_SMD_3225-4Pin_3.2x2.5mm
- added SW10: SW_SK6812MINI-E_Rotated, CherryMX_PCB_LTST-A683CEGBW-Rotated:CherryMX_1.00u_PCB_LTST-A683CEGBW-Rotated, F.Cu at (171.4, 0.00)
- added SW11: SW_SK6812MINI-E_Rotated, CherryMX_PCB_LTST-A683CEGBW-Rotated:CherryMX_1.00u_PCB_LTST-A683CEGBW-Rotated, F.Cu at (190.5, 0.00)
- added SW12: SW_SK6812MINI-E_Rotated, CherryMX_PCB_LTST-A683CEGBW-Rotated:CherryMX_1.00u_PCB_LTST-A683CEGBW-Rotated, F.Cu at (209.6, 0.00)
- added SW13: SW_SK6812MINI-E_Rotated, CherryMX_PCB_LTST-A683CEGBW-Rotated:CherryMX_1.00u_PCB_LTST-A683CEGBW-Rotated, F.Cu at (228.6, 0.00)
- added SW14: SW_SK6812MINI-E_Rotated, CherryMX_PCB_LTST-A683CEGBW-Rotated:CherryMX_1.50u_PCB_LTST-A683CEGBW-Rotated, F.Cu at (252.4, 0.00)
- added SW15: SW_SK6812MINI-E_Rotated, CherryMX_PCB_LTST-A683CEGBW-Rotated:CherryMX_1.00u_PCB_LTST-A683CEGBW-Rotated, F.Cu at (286.9, 0.00)
- added SW16: SW_SK6812MINI-E_Rotated, CherryMX_PCB_LTST-A683CEGBW-Rotated:CherryMX_1.00u_PCB_LTST-A683CEGBW-Rotated, F.Cu at (306.0, 0.00)
- added SW17: SW_SK6812MINI-E_Rotated, CherryMX_PCB_LTST-A683CEGBW-Rotated:CherryMX_1.00u_PCB_LTST-A683CEGBW-Rotated, F.Cu at (325.0, 0.00)
- added SW18: SW_SK6812MINI-E_Rotated, CherryMX_PCB_LTST-A683CEGBW-Rotated:CherryMX_1.00u_PCB_LTST-A683CEGBW-Rotated, F.Cu at (344.1, 0.00)
- added SW19: SW_SK6812MINI-E, CherryMX_PCB_LTST-A683CEGBW:CherryMX_1.50u_PCB_LTST-A683CEGBW, F.Cu at (163.3, 175.2)
- added SW2: SW_SK6812MINI-E_Rotated, CherryMX_PCB_LTST-A683CEGBW-Rotated:CherryMX_1.00u_PCB_LTST-A683CEGBW-Rotated, F.Cu at (19.1, 0.00)
- added SW20: SW_SK6812MINI-E, CherryMX_PCB_LTST-A683CEGBW:CherryMX_1.00u_PCB_LTST-A683CEGBW, F.Cu at (279.8, 54.2)
- added SW21: SW_SK6812MINI-E, CherryMX_PCB_LTST-A683CEGBW:CherryMX_1.00u_PCB_LTST-A683CEGBW, F.Cu at (244.0, 74.4)
- added SW22: SW_SK6812MINI-E, CherryMX_PCB_LTST-A683CEGBW:CherryMX_1.00u_PCB_LTST-A683CEGBW, F.Cu at (223.8, 94.5)
- added SW23: SW_SK6812MINI-E, CherryMX_PCB_LTST-A683CEGBW:CherryMX_1.00u_PCB_LTST-A683CEGBW, F.Cu at (203.7, 114.7)
- added SW24: SW_SK6812MINI-E, CherryMX_PCB_LTST-A683CEGBW:CherryMX_1.00u_PCB_LTST-A683CEGBW, F.Cu at (183.5, 134.9)
- added SW25: SW_SK6812MINI-E, CherryMX_PCB_LTST-A683CEGBW:CherryMX_1.00u_PCB_LTST-A683CEGBW, F.Cu at (163.3, 155.0)
- added SW26: SW_SK6812MINI-E, CherryMX_PCB_LTST-A683CEGBW:CherryMX_1.00u_PCB_LTST-A683CEGBW, F.Cu at (143.2, 175.2)
- added SW27: SW_SK6812MINI-E, CherryMX_PCB_LTST-A683CEGBW:CherryMX_1.00u_PCB_LTST-A683CEGBW, F.Cu at (259.7, 54.2)
- added SW28: SW_SK6812MINI-E, CherryMX_PCB_LTST-A683CEGBW:CherryMX_1.00u_PCB_LTST-A683CEGBW, F.Cu at (223.8, 74.4)
- added SW29: SW_SK6812MINI-E, CherryMX_PCB_LTST-A683CEGBW:CherryMX_1.00u_PCB_LTST-A683CEGBW, F.Cu at (203.7, 94.5)
- added SW3: SW_SK6812MINI-E_Rotated, CherryMX_PCB_LTST-A683CEGBW-Rotated:CherryMX_1.00u_PCB_LTST-A683CEGBW-Rotated, F.Cu at (38.1, 0.00)
- added SW30: SW_SK6812MINI-E, CherryMX_PCB_LTST-A683CEGBW:CherryMX_1.00u_PCB_LTST-A683CEGBW, F.Cu at (183.5, 114.7)
- added SW31: SW_SK6812MINI-E, CherryMX_PCB_LTST-A683CEGBW:CherryMX_1.00u_PCB_LTST-A683CEGBW, F.Cu at (163.3, 134.9)
- added SW32: SW_SK6812MINI-E, CherryMX_PCB_LTST-A683CEGBW:CherryMX_1.00u_PCB_LTST-A683CEGBW, F.Cu at (143.2, 155.0)
- added SW33: SW_SK6812MINI-E, CherryMX_PCB_LTST-A683CEGBW:CherryMX_1.00u_PCB_LTST-A683CEGBW, F.Cu at (123.0, 175.2)
- added SW34: SW_SK6812MINI-E, CherryMX_PCB_LTST-A683CEGBW:CherryMX_1.00u_PCB_LTST-A683CEGBW, F.Cu at (239.5, 54.2)
- added SW35: SW_SK6812MINI-E, CherryMX_PCB_LTST-A683CEGBW:CherryMX_1.00u_PCB_LTST-A683CEGBW, F.Cu at (203.7, 74.4)
- added SW36: SW_SK6812MINI-E, CherryMX_PCB_LTST-A683CEGBW:CherryMX_1.00u_PCB_LTST-A683CEGBW, F.Cu at (183.5, 94.5)
- added SW37: SW_SK6812MINI-E_Rotated, CherryMX_PCB_LTST-A683CEGBW-Rotated:CherryMX_1.75u_PCB_LTST-A683CEGBW-Rotated, F.Cu at (163.3, 114.7)
- added SW38: SW_SK6812MINI-E_Rotated, CherryMX_PCB_LTST-A683CEGBW-Rotated:CherryMX_1.00u_PCB_LTST-A683CEGBW-Rotated, F.Cu at (143.2, 134.9)
- added SW39: SW_SK6812MINI-E_Rotated, CherryMX_PCB_LTST-A683CEGBW-Rotated:CherryMX_1.00u_PCB_LTST-A683CEGBW-Rotated, F.Cu at (123.0, 155.0)
- added SW4: SW_SK6812MINI-E_Rotated, CherryMX_PCB_LTST-A683CEGBW-Rotated:CherryMX_1.00u_PCB_LTST-A683CEGBW-Rotated, F.Cu at (57.1, 0.00)
- added SW40: SW_SK6812MINI-E_Rotated, CherryMX_PCB_LTST-A683CEGBW-Rotated:CherryMX_1.00u_PCB_LTST-A683CEGBW-Rotated, F.Cu at (102.8, 175.2)
- added SW41: SW_SK6812MINI-E_Rotated, CherryMX_PCB_LTST-A683CEGBW-Rotated:CherryMX_1.00u_PCB_LTST-A683CEGBW-Rotated, F.Cu at (219.3, 54.2)
- added SW42: SW_SK6812MINI-E_Rotated, CherryMX_PCB_LTST-A683CEGBW-Rotated:CherryMX_1.00u_PCB_LTST-A683CEGBW-Rotated, F.Cu at (183.5, 74.4)
- added SW43: SW_SK6812MINI-E_Rotated, CherryMX_PCB_LTST-A683CEGBW-Rotated:CherryMX_1.00u_PCB_LTST-A683CEGBW-Rotated, F.Cu at (163.3, 94.5)
- added SW44: SW_SK6812MINI-E_Rotated, CherryMX_PCB_LTST-A683CEGBW-Rotated:CherryMX_1.00u_PCB_LTST-A683CEGBW-Rotated, F.Cu at (143.2, 114.7)
- added SW45: SW_SK6812MINI-E_Rotated, CherryMX_PCB_LTST-A683CEGBW-Rotated:CherryMX_1.00u_PCB_LTST-A683CEGBW-Rotated, F.Cu at (123.0, 134.9)
- added SW46: SW_SK6812MINI-E_Rotated, CherryMX_PCB_LTST-A683CEGBW-Rotated:CherryMX_1.00u_PCB_LTST-A683CEGBW-Rotated, F.Cu at (102.8, 155.0)
- added SW47: SW_SK6812MINI-E_Rotated, CherryMX_PCB_LTST-A683CEGBW-Rotated:CherryMX_1.00u_PCB_LTST-A683CEGBW-Rotated, F.Cu at (82.6, 175.2)
- added SW48: SW_SK6812MINI-E_Rotated, CherryMX_PCB_LTST-A683CEGBW-Rotated:CherryMX_1.00u_PCB_LTST-A683CEGBW-Rotated, F.Cu at (199.2, 54.2)
- added SW49: SW_SK6812MINI-E_Rotated, CherryMX_PCB_LTST-A683CEGBW-Rotated:CherryMX_1.75u_PCB_LTST-A683CEGBW-Rotated, F.Cu at (163.3, 74.4)
- added SW5: SW_SK6812MINI-E_Rotated, CherryMX_PCB_LTST-A683CEGBW-Rotated:CherryMX_1.00u_PCB_LTST-A683CEGBW-Rotated, F.Cu at (76.2, 0.00)
- added SW50: SW_SK6812MINI-E_Rotated, CherryMX_PCB_LTST-A683CEGBW-Rotated:CherryMX_1.00u_PCB_LTST-A683CEGBW-Rotated, F.Cu at (143.2, 94.5)
- added SW51: SW_SK6812MINI-E_Rotated, CherryMX_PCB_LTST-A683CEGBW-Rotated:CherryMX_1.00u_PCB_LTST-A683CEGBW-Rotated, F.Cu at (123.0, 114.7)
- added SW52: SW_SK6812MINI-E_Rotated, CherryMX_PCB_LTST-A683CEGBW-Rotated:CherryMX_1.00u_PCB_LTST-A683CEGBW-Rotated, F.Cu at (102.8, 134.9)
- added SW53: SW_SK6812MINI-E_Rotated, CherryMX_PCB_LTST-A683CEGBW-Rotated:CherryMX_1.00u_PCB_LTST-A683CEGBW-Rotated, F.Cu at (82.6, 155.0)
- added SW54: SW_SK6812MINI-E, CherryMX_PCB_StabWireBottom_LTST-A683CEGBW:CherryMX_2.25u_PCB_StabWireBottom_LTST-A683CEGBW, F.Cu at (62.5, 175.2)
- added SW55: SW_SK6812MINI-E, CherryMX_PCB_LTST-A683CEGBW:CherryMX_1.00u_PCB_LTST-A683CEGBW, F.Cu at (179.0, 54.2)
- added SW56: SW_SK6812MINI-E, CherryMX_PCB_LTST-A683CEGBW:CherryMX_1.00u_PCB_LTST-A683CEGBW, F.Cu at (143.2, 74.4)
- added SW57: SW_SK6812MINI-E, CherryMX_PCB_LTST-A683CEGBW:CherryMX_1.00u_PCB_LTST-A683CEGBW, F.Cu at (123.0, 94.5)
- added SW58: SW_SK6812MINI-E, CherryMX_PCB_LTST-A683CEGBW:CherryMX_1.00u_PCB_LTST-A683CEGBW, F.Cu at (102.8, 114.7)
- added SW59: SW_SK6812MINI-E, CherryMX_PCB_LTST-A683CEGBW:CherryMX_1.00u_PCB_LTST-A683CEGBW, F.Cu at (82.6, 134.9)
- added SW6: SW_SK6812MINI-E_Rotated, CherryMX_PCB_LTST-A683CEGBW-Rotated:CherryMX_1.00u_PCB_LTST-A683CEGBW-Rotated, F.Cu at (95.2, 0.00)
- added SW60: SW_SK6812MINI-E, CherryMX_PCB_LTST-A683CEGBW:CherryMX_1.00u_PCB_LTST-A683CEGBW, F.Cu at (62.5, 155.0)
- added SW61: SW_SK6812MINI-E, CherryMX_PCB_LTST-A683CEGBW:CherryMX_1.00u_PCB_LTST-A683CEGBW, F.Cu at (42.3, 174.2)
- added SW62: SW_SK6812MINI-E, CherryMX_PCB_LTST-A683CEGBW:CherryMX_1.00u_PCB_LTST-A683CEGBW, F.Cu at (158.8, 54.2)
- added SW63: SW_SK6812MINI-E, CherryMX_PCB_LTST-A683CEGBW:CherryMX_1.00u_PCB_LTST-A683CEGBW, F.Cu at (123.0, 74.4)
- added SW64: SW_SK6812MINI-E, CherryMX_PCB_LTST-A683CEGBW:CherryMX_1.00u_PCB_LTST-A683CEGBW, F.Cu at (102.8, 94.5)
- added SW65: SW_SK6812MINI-E, CherryMX_PCB_LTST-A683CEGBW:CherryMX_1.00u_PCB_LTST-A683CEGBW, F.Cu at (82.6, 114.7)
- added SW66: SW_SK6812MINI-E, CherryMX_PCB_StabWireBottom_LTST-A683CEGBW:CherryMX_2.25u_PCB_StabWireBottom_LTST-A683CEGBW, F.Cu at (62.5, 134.9)
- added SW67: SW_SK6812MINI-E, CherryMX_PCB_LTST-A683CEGBW:CherryMX_1.00u_PCB_LTST-A683CEGBW, F.Cu at (42.3, 154.0)
- added SW68: SW_SK6812MINI-E, CherryMX_PCB_LTST-A683CEGBW:CherryMX_1.00u_PCB_LTST-A683CEGBW, F.Cu at (138.6, 54.2)
- added SW69: SW_SK6812MINI-E, CherryMX_PCB_LTST-A683CEGBW:CherryMX_1.00u_PCB_LTST-A683CEGBW, F.Cu at (102.8, 74.4)
- added SW7: SW_SK6812MINI-E_Rotated, CherryMX_PCB_LTST-A683CEGBW-Rotated:CherryMX_1.00u_PCB_LTST-A683CEGBW-Rotated, F.Cu at (114.3, 0.00)
- added SW70: SW_SK6812MINI-E_Rotated, CherryMX_PCB_LTST-A683CEGBW-Rotated:CherryMX_1.50u_PCB_LTST-A683CEGBW-Rotated, F.Cu at (82.6, 94.5)
- added SW71: SW_SK6812MINI-E_Rotated, CherryMX_PCB_StabWireBottom_LTST-A683CEGBW-Rotated:CherryMX_2.00u_PCB_StabWireBottom_LTST-A683CEGBW-Rotated, F.Cu at (62.5, 114.7)
- added SW72: SW_SK6812MINI-E_Rotated, CherryMX_PCB_StabWireBottom_LTST-A683CEGBW-Rotated:CherryMX_7.00u_PCB_StabWireBottom_LTST-A683CEGBW-Rotated, F.Cu at (42.3, 133.9)
- added SW73: SW_SK6812MINI-E_Rotated, CherryMX_PCB_LTST-A683CEGBW-Rotated:CherryMX_1.00u_PCB_LTST-A683CEGBW-Rotated, F.Cu at (118.5, 54.2)
- added SW74: SW_SK6812MINI-E_Rotated, CherryMX_PCB_LTST-A683CEGBW-Rotated:CherryMX_1.00u_PCB_LTST-A683CEGBW-Rotated, F.Cu at (82.6, 74.4)
- added SW75: SW_SK6812MINI-E_Rotated, CherryMX_PCB_LTST-A683CEGBW-Rotated:CherryMX_1.00u_PCB_LTST-A683CEGBW-Rotated, F.Cu at (62.5, 94.5)
- added SW76: SW_SK6812MINI-E_Rotated, CherryMX_PCB_LTST-A683CEGBW-Rotated:CherryMX_1.00u_PCB_LTST-A683CEGBW-Rotated, F.Cu at (42.3, 113.7)
- added SW77: SW_SK6812MINI-E_Rotated, CherryMX_PCB_StabWireBottom_LTST-A683CEGBW-Rotated:CherryMX_2.00u_PCB_StabWireBottom_LTST-A683CEGBW-Rotated, F.Cu at (98.3, 54.2)
- added SW78: SW_SK6812MINI-E_Rotated, CherryMX_PCB_LTST-A683CEGBW-Rotated:CherryMX_1.00u_PCB_LTST-A683CEGBW-Rotated, F.Cu at (62.5, 74.4)
- added SW79: SW_SK6812MINI-E_Rotated, CherryMX_PCB_StabWireBottom_LTST-A683CEGBW-Rotated:CherryMX_2.00u_PCB_StabWireBottom_LTST-A683CEGBW-Rotated, F.Cu at (42.3, 93.5)
- added SW8: SW_SK6812MINI-E_Rotated, CherryMX_PCB_LTST-A683CEGBW-Rotated:CherryMX_1.00u_PCB_LTST-A683CEGBW-Rotated, F.Cu at (133.3, 0.00)
- added SW9: SW_SK6812MINI-E_Rotated, CherryMX_PCB_LTST-A683CEGBW-Rotated:CherryMX_1.00u_PCB_LTST-A683CEGBW-Rotated, F.Cu at (152.4, 0.00)
- D1, D10, D11, D12, D13, D14, D15, D16, D17, D18, D19, D2, D20, D21, D22, D23, D24, D25, D26, D27, D28, D29, D3, D30, D31, D32, D33, D34, D35, D36, D37, D38, D39, D4, D40, D41, D42, D43, D44, D45, D46, D47, D48, D49, D5, D50, D51, D52, D53, D54, D55, D56, D57, D58, D59, D6, D60, D61, D62, D63, D64, D65, D66, D67, D68, D69, D7, D70, D71, D72, D73, D74, D75, D76, D77, D78, D79, D8, D9: footprint Diode_SMD:D_SOD-123 -> Keebio-Parts:Diode; moved to F.Cu
- SW1: value SW_Push -> SW_SK6812MINI-E_Rotated; footprint random-keyboard-parts:SKQG-1155865 -> CherryMX_PCB_LTST-A683CEGBW-Rotated:CherryMX_1.00u_PCB_LTST-A683CEGBW-Rotated; moved to F.Cu
- U1: value ATmega32U4-AU -> Elite-C; footprint Package_QFP:TQFP-44_10x10mm_P0.8mm -> Keebio-Parts:Elite-C; moved to F.Cu
- moved D69 318.0 mm to (47.6, 197.5), turned to 0 degrees
- moved D70 312.3 mm to (57.9, 194.0), turned to 0 degrees
- moved D53 307.7 mm to (88.7, 197.5), turned to 0 degrees
- moved D68 291.9 mm to (57.9, 197.5), turned to 0 degrees
- moved D1 291.3 mm to (279.4, 106.4), turned to 0 degrees
- moved D73 287.8 mm to (68.2, 187.0), turned to 0 degrees
- moved D52 283.0 mm to (99.0, 197.5), turned to 0 degrees
- moved D72 282.7 mm to (57.9, 190.5), turned to 0 degrees
- moved D36 276.9 mm to (140.1, 197.5), turned to 0 degrees
- moved D67 264.7 mm to (68.2, 194.0), turned to 0 degrees
- moved D51 257.1 mm to (109.2, 194.0), turned to 0 degrees
- moved D71 256.2 mm to (68.2, 190.5), turned to 0 degrees
- moved D21 247.8 mm to (299.6, 63.3), turned to 0 degrees
- moved D16 243.4 mm to (170.9, 197.5), turned to 0 degrees
- moved D19 239.8 mm to (181.1, 190.5), turned to 0 degrees
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Connections:
- D70 pad 1: ROW3 -> ROW4
- SW1 pad 1: GND -> COL0
- SW1 pad 2: Net-(R1-Pad2) -> Net-(D1-Pad2)
- SW1 pad 3: (no net) -> VCC
- SW1 pad 4: (no net) -> Net-(SW1-Pad4)
- U1 pad 1: Net-(U1-Pad1) -> LED
- U1 pad 13: Net-(R1-Pad2) -> Net-(U1-Pad13)
- U1 pad 14: +5V -> Net-(U1-Pad14)
- U1 pad 15: GND -> Net-(U1-Pad15)
- U1 pad 2: +5V -> Net-(U1-Pad2)
- U1 pad 21: Net-(U1-Pad21) -> VCC
- U1 pad 24: +5V -> Net-(U1-Pad24)
- U1 pad 3: Net-(R3-Pad1) -> GND
- U1 pad 4: Net-(R2-Pad1) -> GND
- U1 pad 5: GND -> Net-(U1-Pad5)
- U1 pad 7: +5V -> Net-(U1-Pad7)
Other:
- board outline added: 3.4 x 3 mm

Commit message: place footprints and connect leds
Parts:
- D1, D10, D11, D12, D13, D14, D15, D16, D17, D18, D19, D2, D20, D21, D22, D23, D24, D25, D26, D27, D28, D29, D3, D30, D31, D32, D33, D34, D35, D36, D37, D38, D39, D4, D40, D41, D42, D43, D44, D45, D46, D47, D48, D49, D5, D50, D51, D52, D53, D54, D55, D56, D57, D58, D59, D6, D60, D61, D62, D63, D64, D65, D66, D67, D68, D69, D7, D70, D71, D72, D73, D74, D75, D76, D77, D78, D79, D8, D9: footprint Keebio-Parts:Diode -> m0110a:Diode; moved to B.Cu
- SW1, SW10, SW11, SW12, SW13, SW15, SW16, SW17, SW18, SW2, SW3, SW38, SW39, SW4, SW40, SW41, SW42, SW43, SW44, SW45, SW46, SW47, SW48, SW5, SW50, SW51, SW52, SW53, SW6, SW7, SW73, SW74, SW75, SW76, SW78, SW8, SW9: footprint CherryMX_PCB_LTST-A683CEGBW-Rotated:CherryMX_1.00u_PCB_LTST-A683CEGBW-Rotated -> CherryMX_PCB_KailhSocket_LTST-A683CEGBW-Rotated:CherryMX_1.00u_PCB_KailhSocket_LTST-A683CEGBW-Rotated
- SW14: footprint CherryMX_PCB_LTST-A683CEGBW-Rotated:CherryMX_1.50u_PCB_LTST-A683CEGBW-Rotated -> CherryMX_PCB_KailhSocket_LTST-A683CEGBW-Rotated:CherryMX_1.50u_PCB_KailhSocket_LTST-A683CEGBW-Rotated
- SW19: footprint CherryMX_PCB_LTST-A683CEGBW:CherryMX_1.50u_PCB_LTST-A683CEGBW -> CherryMX_PCB_KailhSocket_LTST-A683CEGBW:CherryMX_1.50u_PCB_KailhSocket_LTST-A683CEGBW
- SW20, SW21, SW22, SW23, SW24, SW25, SW26, SW27, SW28, SW29, SW30, SW31, SW32, SW33, SW34, SW35, SW36, SW55, SW56, SW57, SW58, SW59, SW60, SW61, SW62, SW63, SW64, SW67, SW68, SW69: footprint CherryMX_PCB_LTST-A683CEGBW:CherryMX_1.00u_PCB_LTST-A683CEGBW -> CherryMX_PCB_KailhSocket_LTST-A683CEGBW:CherryMX_1.00u_PCB_KailhSocket_LTST-A683CEGBW
- SW37, SW49: footprint CherryMX_PCB_LTST-A683CEGBW-Rotated:CherryMX_1.75u_PCB_LTST-A683CEGBW-Rotated -> CherryMX_PCB_KailhSocket_LTST-A683CEGBW-Rotated:CherryMX_1.75u_PCB_KailhSocket_LTST-A683CEGBW-Rotated
- SW54: footprint CherryMX_PCB_StabWireBottom_LTST-A683CEGBW:CherryMX_2.25u_PCB_StabWireBottom_LTST-A683CEGBW -> CherryMX_PCB_KailhSocket_StabWireBottom_LTST-A683CEGBW:CherryMX_2.25u_PCB_KailhSocket_StabWireBottom_LTST-A683CEGBW
- SW65: footprint CherryMX_PCB_LTST-A683CEGBW:CherryMX_1.00u_PCB_LTST-A683CEGBW -> CherryMX_PCB_KailhSocket_LTST-A683CEGBW:CherryMX_1.25u_PCB_KailhSocket_LTST-A683CEGBW
- SW66: footprint CherryMX_PCB_StabWireBottom_LTST-A683CEGBW:CherryMX_2.25u_PCB_StabWireBottom_LTST-A683CEGBW -> CherryMX_PCB_KailhSocket_LTST-A683CEGBW:CherryMX_1.00u_PCB_KailhSocket_LTST-A683CEGBW
- SW70: footprint CherryMX_PCB_LTST-A683CEGBW-Rotated:CherryMX_1.50u_PCB_LTST-A683CEGBW-Rotated -> CherryMX_PCB_KailhSocket_LTST-A683CEGBW:CherryMX_1.50u_PCB_KailhSocket_LTST-A683CEGBW
- SW71, SW77, SW79: footprint CherryMX_PCB_StabWireBottom_LTST-A683CEGBW-Rotated:CherryMX_2.00u_PCB_StabWireBottom_LTST-A683CEGBW-Rotated -> CherryMX_PCB_KailhSocket_StabWireBottom_LTST-A683CEGBW-Rotated:CherryMX_2.00u_PCB_KailhSocket_StabWireBottom_LTST-A683C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
- SW72: footprint CherryMX_PCB_StabWireBottom_LTST-A683CEGBW-Rotated:CherryMX_7.00u_PCB_StabWireBottom_LTST-A683CEGBW-Rotated -> CherryMX_PCB_KailhSocket_StabWireBottom_LTST-A683CEGBW-Rotated:CherryMX_7.00u_PCB_KailhSocket_StabWireBottom_LTST-A683C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
- moved D69 319.1 mm to (333.6, 55.9), turned to 270 degrees
- moved D53 309.1 mm to (352.8, 36.8), turned to 270 degrees
- moved D78 308.5 mm to (333.6, 74.9), turned to 270 degrees
- moved D79 308.1 mm to (337.4, 82.4), turned to 180 degrees
- moved SW79 302.9 mm to (344.1, 66.7), turned to 90 degrees
- moved D68 293.1 mm to (314.6, 55.9), turned to 270 degrees
- moved D77 292.7 mm to (305.2, 74.9), turned to 270 degrees
- moved D1 291.4 mm to (8.64, -1.27), turned to 270 degrees
- moved SW53 286.4 mm to (344.1, 38.1)
- moved D52 284.5 mm to (333.8, 36.8), turned to 270 degrees
- moved D36 278.4 mm to (352.7, 17.8), turned to 270 degrees
- moved D67 266.0 mm to (295.5, 55.9), turned to 270 degrees
- moved SW67 263.1 mm to (286.9, 57.1)
- moved SW78 262.5 mm to (325.0, 76.2)
- moved D76 258.8 mm to (265.8, 74.9), turned to 270 degrees
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Connections:
- U1 pad 26: Net-(U1-Pad26) -> ROW4
Routing:
- net ROW0: track 0.00 -> 344.0 mm
- net ROW1: track 0.00 -> 339.2 mm
- net ROW2: track 0.00 -> 336.7 mm
- net ROW4: track 0.00 -> 323.9 mm
- net ROW3: track 0.00 -> 313.1 mm
- net COL9: track 0.00 -> 91.2 mm
- net COL11: track 0.00 -> 90.0 mm
- net COL12: track 0.00 -> 88.9 mm
- net COL5: track 0.00 -> 88.8 mm
- net COL10: track 0.00 -> 88.8 mm
- net COL1: track 0.00 -> 88.1 mm
- net COL0: track 0.00 -> 85.9 mm
- net COL14: track 0.00 -> 83.3 mm
- net COL17: track 0.00 -> 81.8 mm
- net COL16: track 0.00 -> 76.2 mm
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- added copper zone on B.Cu, net GND
Other:
- board size 3.4 x 3 mm -> 3 x 3.4 mm
- net class Default: trace_width 0.25 -> 0.254
- net class Power added: clearance 0.2, trace_width 0.381, via_dia 0.8, via_drill 0.4

Commit message: start connecting VCC
Parts:
- U1: moved to B.Cu
Connections:
- U1 pad 26: ROW4 -> Net-(U1-Pad26)
- U1 pad 28: Net-(U1-Pad28) -> ROW4
Routing:
- net Net-(SW71-Pad4): track 0.00 -> 85.5 mm
- net VCC: track 0.00 -> 21.5 mm

Commit message: first complete pcb
Parts:
- moved D18 2.13 mm to (354.8, -1.27)
- moved D77 2.03 mm to (307.2, 74.9)
- moved D69 2.03 mm to (335.7, 55.9)
- moved D78 1.80 mm to (335.4, 74.7)
- moved D33 1.78 mm to (297.3, 17.8)
- moved D67 1.78 mm to (297.3, 55.9)
- moved SW77 1.71 mm to (298.1, 76.2)
- moved SW16 1.70 mm to (307.7, 0.00)
- moved SW34 1.70 mm to (307.7, 19.1)
- moved SW51 1.70 mm to (307.7, 38.1)
- moved SW68 1.70 mm to (307.7, 57.1)
- moved SW15 1.70 mm to (288.6, 0.00)
- moved SW17 1.70 mm to (326.7, 0.00)
- moved SW18 1.70 mm to (345.8, 0.00)
- moved SW33 1.70 mm to (288.6, 19.1)
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Connections:
- SW43 pad 3: Net-(SW43-Pad3) -> VCC
- SW61 pad 3: Net-(SW61-Pad3) -> VCC
- SW79 pad 1: COL17 -> Net-(D79-Pad2)
- SW79 pad 2: Net-(D79-Pad2) -> COL17
- U1 pad 10: Net-(U1-Pad10) -> COL10
- U1 pad 11: Net-(U1-Pad11) -> COL11
- U1 pad 12: Net-(U1-Pad12) -> COL13
- U1 pad 13: Net-(U1-Pad13) -> COL16
- U1 pad 14: Net-(U1-Pad14) -> COL17
- U1 pad 15: Net-(U1-Pad15) -> ROW0
- U1 pad 16: Net-(U1-Pad16) -> ROW1
- U1 pad 17: Net-(U1-Pad17) -> ROW2
- U1 pad 18: Net-(U1-Pad18) -> COL3
- U1 pad 19: Net-(U1-Pad19) -> COL2
- U1 pad 2: Net-(U1-Pad2) -> ROW3
- U1 pad 20: Net-(U1-Pad20) -> COL0
- U1 pad 24: Net-(U1-Pad24) -> COL1
- U1 pad 25: Net-(U1-Pad25) -> COL12
- U1 pad 26: Net-(U1-Pad26) -> COL5
- U1 pad 27: Net-(U1-Pad27) -> ROW4
- U1 pad 28: ROW4 -> COL14
- U1 pad 29: Net-(U1-Pad29) -> COL15
- U1 pad 5: Net-(U1-Pad5) -> COL4
- U1 pad 6: Net-(U1-Pad6) -> COL6
- U1 pad 7: Net-(U1-Pad7) -> COL7
- U1 pad 8: Net-(U1-Pad8) -> COL8
- U1 pad 9: Net-(U1-Pad9) -> COL9
Routing:
- net VCC: track 21.5 -> 2102.9 mm, vias 0 -> 72
- net COL17: track 81.8 -> 350.0 mm, vias 0 -> 1
- net COL13: track 21.0 -> 245.6 mm, vias 0 -> 1
- net COL16: track 76.2 -> 299.3 mm, vias 0 -> 1
- net COL15: track 57.1 -> 274.7 mm, vias 0 -> 3
- net COL14: track 83.3 -> 268.9 mm, vias 0 -> 1
- net ROW0: track 344.0 -> 504.5 mm, vias 0 -> 8
- net COL12: track 88.9 -> 234.1 mm, vias 0 -> 1
- net ROW1: track 339.2 -> 479.0 mm, vias 0 -> 6
- net COL11: track 90.0 -> 215.0 mm, vias 0 -> 1
- net COL0: track 85.9 -> 196.8 mm, vias 0 -> 2
- net COL10: track 88.8 -> 194.1 mm, vias 0 -> 1
- net COL9: track 91.2 -> 178.4 mm, vias 0 -> 1
- net LED: track 0.00 -> 81.0 mm, vias 0 -> 1
- net COL8: track 67.0 -> 145.4 mm, vias 0 -> 1
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Other:
- board size 3 x 3.4 mm -> 2.4 x 97.6 mm

Commit message: Fix DRC errors
Routing:
- net COL17: track 350.0 -> 354.8 mm
- net VCC: track 2102.9 -> 2102.0 mm
- net COL15: track 274.7 -> 273.7 mm
Other:
- board size 2.4 x 97.6 mm -> 367.5 x 96.8 mm
