File: m0110a.kicad_pcb (KiCad board)
At the start: 2 copper layers, 367.5 x 96.8 mm, 159 parts, among them SW1 SW_SK6812MINI-E_Rotated, SW10 SW_SK6812MINI-E_Rotated, SW11 SW_SK6812MINI-E_Rotated, SW12 SW_SK6812MINI-E_Rotated, SW13 SW_SK6812MINI-E_Rotated, SW14 SW_SK6812MINI-E_Rotated, SW15 SW_SK6812MINI-E_Rotated, SW16 SW_SK6812MINI-E_Rotated, SW17 SW_SK6812MINI-E_Rotated, SW18 SW_SK6812MINI-E_Rotated, SW19 SW_SK6812MINI-E, SW2 SW_SK6812MINI-E_Rotated, SW20 SW_SK6812MINI-E, SW21 SW_SK6812MINI-E, SW22 SW_SK6812MINI-E, SW23 SW_SK6812MINI-E, SW24 SW_SK6812MINI-E, SW25 SW_SK6812MINI-E, SW26 SW_SK6812MINI-E, SW27 SW_SK6812MINI-E, SW28 SW_SK6812MINI-E, SW29 SW_SK6812MINI-E, SW3 SW_SK6812MINI-E_Rotated, SW30 SW_SK6812MINI-E, SW31 SW_SK6812MINI-E, SW32 SW_SK6812MINI-E, SW33 SW_SK6812MINI-E, SW34 SW_SK6812MINI-E, SW35 SW_SK6812MINI-E, SW36 SW_SK6812MINI-E, SW37 SW_SK6812MINI-E_Rotated, SW38 SW_SK6812MINI-E_Rotated, SW39 SW_SK6812MINI-E_Rotated, SW4 SW_SK6812MINI-E_Rotated, SW40 SW_SK6812MINI-E_Rotated, SW41 SW_SK6812MINI-E_Rotated, SW42 SW_SK6812MINI-E_Rotated, SW43 SW_SK6812MINI-E_Rotated, SW44 SW_SK6812MINI-E_Rotated, SW45 SW_SK6812MINI-E_Rotated, SW46 SW_SK6812MINI-E_Rotated, SW47 SW_SK6812MINI-E_Rotated, SW48 SW_SK6812MINI-E_Rotated, SW49 SW_SK6812MINI-E_Rotated, SW5 SW_SK6812MINI-E_Rotated, SW50 SW_SK6812MINI-E_Rotated, SW51 SW_SK6812MINI-E_Rotated, SW52 SW_SK6812MINI-E_Rotated, SW53 SW_SK6812MINI-E_Rotated, SW54 SW_SK6812MINI-E, SW55 SW_SK6812MINI-E, SW56 SW_SK6812MINI-E, SW57 SW_SK6812MINI-E, SW58 SW_SK6812MINI-E, SW59 SW_SK6812MINI-E, SW6 SW_SK6812MINI-E_Rotated, SW60 SW_SK6812MINI-E, SW61 SW_SK6812MINI-E, SW62 SW_SK6812MINI-E, SW63 SW_SK6812MINI-E, SW64 SW_SK6812MINI-E, SW65 SW_SK6812MINI-E, SW66 SW_SK6812MINI-E, SW67 SW_SK6812MINI-E, SW68 SW_SK6812MINI-E, SW69 SW_SK6812MINI-E, SW7 SW_SK6812MINI-E_Rotated, SW70 SW_SK6812MINI-E_Rotated, SW71 SW_SK6812MINI-E_Rotated, SW72 SW_SK6812MINI-E_Rotated, SW73 SW_SK6812MINI-E_Rotated, SW74 SW_SK6812MINI-E_Rotated, SW75 SW_SK6812MINI-E_Rotated, SW76 SW_SK6812MINI-E_Rotated, SW77 SW_SK6812MINI-E_Rotated, SW78 SW_SK6812MINI-E_Rotated, SW79 SW_SK6812MINI-E_Rotated, SW8 SW_SK6812MINI-E_Rotated, SW9 SW_SK6812MINI-E_Rotated, U1 Elite-C

Commit message: add row, led data and vcc tracks start columns
Parts:
- moved D79 1.78 mm to (339.2, 82.4)
Routing:
- net COL17: track 354.8 -> 65.1 mm, vias 1 -> 6
- net COL15: track 273.7 -> 0.00 mm, vias 3 -> 0
- net COL14: track 268.7 -> 0.00 mm, vias 1 -> 0
- net COL12: track 234.1 -> 0.00 mm, vias 1 -> 0
- net COL13: track 245.6 -> 21.0 mm, vias 1 -> 2
- net COL16: track 299.2 -> 76.6 mm, vias 1 -> 8
- net COL11: track 215.0 -> 0.00 mm, vias 1 -> 0
- net VCC: track 2102.1 -> 1901.4 mm, vias 72 -> 3
- net ROW0: track 545.3 -> 346.2 mm, vias 1 -> 0
- net COL10: track 194.1 -> 0.00 mm, vias 1 -> 0
- net COL9: track 178.4 -> 0.00 mm, vias 1 -> 0
- net ROW1: track 519.4 -> 371.5 mm, vias 1 -> 0
- net COL1: track 146.4 -> 0.00 mm
- net COL8: track 145.4 -> 0.00 mm, vias 1 -> 0
- net COL2: track 133.8 -> 0.00 mm, vias 2 -> 0
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
Commit message: horiontal done
Routing:
- net COL17: track 65.1 -> 356.5 mm
- net COL15: track 0.00 -> 270.4 mm, vias 0 -> 9
- net COL14: track 0.00 -> 269.5 mm, vias 0 -> 10
- net COL12: track 0.00 -> 235.4 mm, vias 0 -> 12
- net COL16: track 76.6 -> 300.4 mm, vias 8 -> 10
- net COL13: track 21.0 -> 243.0 mm, vias 2 -> 13
- net COL11: track 0.00 -> 220.4 mm, vias 0 -> 10
- net COL10: track 0.00 -> 202.5 mm, vias 0 -> 8
- net ROW0: track 346.2 -> 544.4 mm, vias 0 -> 3
- net COL9: track 0.00 -> 184.6 mm, vias 0 -> 8
- net COL8: track 0.00 -> 148.1 mm, vias 0 -> 7
- net COL1: track 0.00 -> 147.3 mm, vias 0 -> 9
- net ROW1: track 371.5 -> 505.0 mm, vias 0 -> 5
- net COL7: track 0.00 -> 131.2 mm, vias 0 -> 7
- net COL2: track 0.00 -> 127.0 mm, vias 0 -> 8
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