File: m0110a.sch (KiCad schematic (older format))
At the start: 159 parts, among them SW1 SW_SK6812MINI-E_Rotated, SW10 SW_SK6812MINI-E_Rotated, SW11 SW_SK6812MINI-E_Rotated, SW12 SW_SK6812MINI-E_Rotated, SW13 SW_SK6812MINI-E_Rotated, SW14 SW_SK6812MINI-E_Rotated, SW15 SW_SK6812MINI-E_Rotated, SW16 SW_SK6812MINI-E_Rotated, SW17 SW_SK6812MINI-E_Rotated, SW18 SW_SK6812MINI-E_Rotated, SW19 SW_SK6812MINI-E, SW2 SW_SK6812MINI-E_Rotated, SW20 SW_SK6812MINI-E, SW21 SW_SK6812MINI-E, SW22 SW_SK6812MINI-E, SW23 SW_SK6812MINI-E, SW24 SW_SK6812MINI-E, SW25 SW_SK6812MINI-E, SW26 SW_SK6812MINI-E, SW27 SW_SK6812MINI-E, SW28 SW_SK6812MINI-E, SW29 SW_SK6812MINI-E, SW3 SW_SK6812MINI-E_Rotated, SW30 SW_SK6812MINI-E, SW31 SW_SK6812MINI-E, SW32 SW_SK6812MINI-E, SW33 SW_SK6812MINI-E, SW34 SW_SK6812MINI-E, SW35 SW_SK6812MINI-E, SW36 SW_SK6812MINI-E, SW37 SW_SK6812MINI-E_Rotated, SW38 SW_SK6812MINI-E_Rotated, SW39 SW_SK6812MINI-E_Rotated, SW4 SW_SK6812MINI-E_Rotated, SW40 SW_SK6812MINI-E_Rotated, SW41 SW_SK6812MINI-E_Rotated, SW42 SW_SK6812MINI-E_Rotated, SW43 SW_SK6812MINI-E_Rotated, SW44 SW_SK6812MINI-E_Rotated, SW45 SW_SK6812MINI-E_Rotated, SW46 SW_SK6812MINI-E_Rotated, SW47 SW_SK6812MINI-E_Rotated, SW48 SW_SK6812MINI-E_Rotated, SW49 SW_SK6812MINI-E_Rotated, SW5 SW_SK6812MINI-E_Rotated, SW50 SW_SK6812MINI-E_Rotated, SW51 SW_SK6812MINI-E_Rotated, SW52 SW_SK6812MINI-E_Rotated, SW53 SW_SK6812MINI-E_Rotated, SW54 SW_SK6812MINI-E, SW55 SW_SK6812MINI-E, SW56 SW_SK6812MINI-E, SW57 SW_SK6812MINI-E, SW58 SW_SK6812MINI-E, SW59 SW_SK6812MINI-E, SW6 SW_SK6812MINI-E_Rotated, SW60 SW_SK6812MINI-E, SW61 SW_SK6812MINI-E, SW62 SW_SK6812MINI-E, SW63 SW_SK6812MINI-E, SW64 SW_SK6812MINI-E, SW65 SW_SK6812MINI-E, SW66 SW_SK6812MINI-E, SW67 SW_SK6812MINI-E, SW68 SW_SK6812MINI-E, SW69 SW_SK6812MINI-E, SW7 SW_SK6812MINI-E_Rotated, SW70 SW_SK6812MINI-E_Rotated, SW71 SW_SK6812MINI-E_Rotated, SW72 SW_SK6812MINI-E_Rotated, SW73 SW_SK6812MINI-E_Rotated, SW74 SW_SK6812MINI-E_Rotated, SW75 SW_SK6812MINI-E_Rotated, SW76 SW_SK6812MINI-E_Rotated, SW77 SW_SK6812MINI-E_Rotated, SW78 SW_SK6812MINI-E_Rotated, SW79 SW_SK6812MINI-E_Rotated, SW8 SW_SK6812MINI-E_Rotated, SW9 SW_SK6812MINI-E_Rotated, U1 Elite-C

Commit message: first complete pcb
Connections:
- wire segments 849 -> 855
Other:
- moved on the sheet: D79
Changed lines of the file:
@@
 $EndDescr
 $Comp
-L keebio:Elite-C U1
-U 1 1 5F5257EF
-P 2670 2330
-F 0 "U1" H 2670 3167 60  0000 C CNN
-F 1 "Elite-C" H 2670 3061 60  0000 C CNN
-F 2 "Keebio-Parts:Elite-C" V 3720 -170 60  0001 C CNN
-F 3 "" V 3720 -170 60  0001 C CNN
-	1    2670 2330
-	1    0    0    -1
-$EndComp
-$Comp
 L power:GND #PWR04
 U 1 1 5F5282F6
@@
 L Device:D_Small D79
 U 1 1 5F6205C8
-P 21570 4930
-F 0 "D79" V 21549 4998 30  0000 L CNN
-F 1 "D_Small" V 21600 4998 20  0000 L CNN
-F 2 "m0110a:Diode" V 21570 4930 50  0001 C CNN
-F 3 "~" V 21570 4930 50  0001 C CNN
-	1    21570 4930
+P 20970 4930
+F 0 "D79" V 20949 4998 30  0000 L CNN
+F 1 "D_Small" V 21000 4998 20  0000 L CNN
+F 2 "m0110a:Diode" V 20970 4930 50  0001 C CNN
+F 3 "~" V 20970 4930 50  0001 C CNN
+	1    20970 4930
 	0    1    1    0
 $EndComp
@@
 Connection ~ 20590 4830
 Wire Wire Line
-	20590 4830 21570 4830
+	20590 4830 20970 4830
 Connection ~ 13820 4830
 Wire Wire Line
@@
 Connection ~ 19940 4010
 Wire Wire Line
-	20970 5030 20930 5030
-Wire Wire Line
-	20930 5030 20930 2960
-Wire Wire Line
 	20930 1000 20960 1000
 Text GLabel 20930 1000 0    50   Input ~ 0
@@
 Wire Wire Line
 	20970 2960 20930 2960
-Connection ~ 20930 2960
 Wire Wire Line
 	20930 2960 20930 1930
@@
 Connection ~ 10210 3420
 Wire Wire Line
-	10210 3420 11830 3420
+	10210 3420 10850 3420
 Wire Wire Line
 	9880 3160 9880 3420
@@
 	21570 5460 21570 5230
 Connection ~ 20590 5460
-Text GLabel 2770 3280 3    50   Input ~ 0
+Text GLabel 2670 3280 3    50   Input ~ 0
 ROW4
+$Comp
+L keebio:Elite-C U1
+U 1 1 5F5257EF
+P 2670 2330
+F 0 "U1" H 2670 3167 60  0000 C CNN
+F 1 "Elite-C" H 2670 3061 60  0000 C CNN
+F 2 "Keebio-Parts:Elite-C" V 3720 -170 60  0001 C CNN
+F 3 "" V 3720 -170 60  0001 C CNN
+	1    2670 2330
+	1    0    0    -1
+$EndComp
+Text GLabel 2570 3280 3    50   Input ~ 0
+COL5
+Text GLabel 1970 1880 0    50   Input ~ 0
+ROW3
+Text GLabel 3370 2480 2    50   Input ~ 0
+ROW2
+Text GLabel 3370 2580 2    50   Input ~ 0
+ROW1
+Text GLabel 3370 2680 2    50   Input ~ 0
+ROW0
+Text GLabel 3370 2180 2    50   Input ~ 0
+COL0
+Text GLabel 3370 1780 2    50   Input ~ 0
+COL1
+Text GLabel 3370 2280 2    50   Input ~ 0
+COL2
+Text GLabel 3370 2380 2    50   Input ~ 0
+COL3
+Text GLabel 1970 2180 0    50   Input ~ 0
+COL4
+Text GLabel 1970 2280 0    50   Input ~ 0
+COL6
+Wire Wire Line
+	21570 3600 20930 3600
+Wire Wire Line
+	20930 3600 20930 2960
+Wire Wire Line
+	21570 3600 21570 5030
+Connection ~ 20930 2960
+Wire Wire Line
+	10850 3160 10850 3420
+Connection ~ 10850 3420
+Wire Wire Line
+	10850 3420 11190 3420
+Wire Wire Line
+	11240 4110 11190 4110
+Wire Wire Line
+	11190 4110 11190 3420
+Connection ~ 11190 3420
+Wire Wire Line
+	11190 3420 11830 3420
+Text GLabel 1970 2380 0    50   Input ~ 0
+COL7
+Text GLabel 1970 2480 0    50   Input ~ 0
+COL8
+Text GLabel 1970 2580 0    50   Input ~ 0
+COL9
+Text GLabel 1970 2680 0    50   Input ~ 0
+COL10
+Text GLabel 1970 2780 0    50   Input ~ 0
+COL11
+Text GLabel 2470 3280 3    50   Input ~ 0
+COL12
+Text GLabel 1970 2880 0    50   Input ~ 0
+COL13
+Text GLabel 2770 3280 3    50   Input ~ 0
+COL14
+Text GLabel 3370 2780 2    50   Input ~ 0
+COL17
+Text GLabel 3370 2880 2    50   Input ~ 0
+COL16
+Text GLabel 2870 3280 3    50   Input ~ 0
+COL15
 $EndSCHEMATC

Commit message: fix row 0 and row 1 tracks
Changed lines of the file:
@@
 Text GLabel 3370 2480 2    50   Input ~ 0
 ROW2
+Text GLabel 3370 2680 2    50   Input ~ 0
+ROW1
 Text GLabel 3370 2580 2    50   Input ~ 0
-ROW1
-Text GLabel 3370 2680 2    50   Input ~ 0
 ROW0
 Text GLabel 3370 2180 2    50   Input ~ 0
